File: woerdclcock.sch (KiCad schematic (older format))
At the start: 46 parts, among them K1 Sound, K2 IR, K3 CONN_3, P1 Jumper, P2 KEY1, P3 KEY2, SW1 up, SW2 ok, SW3 down, U1 HOHLSTECKER, U10 DCF77, U11 DHT, U12 WS2811, U13 WS2811, U14 SD-CARD, U2 RTC_MODUL, U3 ARDUINO_MINI_PRO, U4 WS2811, U6 HC-05, U7 HC-05, U8 ESP8266, U9 10DOF

Commit message: first commit
Parts:
- removed P2: KEY1, symbol CONN_1
- removed P3: KEY2, symbol CONN_1
- removed U1: HOHLSTECKER, symbol HOHLSTECKER
- removed U12, U13, U4: WS2811, symbol WS2811
- added C2, C3: 0,1uF, symbol C
- added K4: CONN_3, symbol CONN_3
- added P2, P3: Jumper, symbol CONN_2
- added P4, P5, P6, P7: CONN_1, symbol CONN_1
- added U1: RFM12B, symbol RFM12B
Connections:
- wire segments 89 -> 63
- no-connect marks 14 -> 19
Other:
- note added: "RFM12b"
- moved on the sheet: D3, D4, K3, R10, R11, R9, U11, U7, U8
